File: Cannula_mother.sch (EAGLE design)
At the start: 82 parts, among them M1 LED_R, M2 LED_R, M3 LED_R, M4 LED_R, M5 LED_R, M6 LED_R, Y1 25 MHZ

Commit message: Changes almost finished
Parts:
- removed ENABLE_GLOBAL: LED_R, Cannula_1_0:LED-0805
- removed TP10: PTR1TP20R, testpad:PTR1TP20R
- added ERROR: LED_G, Cannula_1_0:LED-0805
- added INHIBIT: LED_R, Cannula_1_0:LED-0805
- added Q1: (no value), adafruit:MOSFET-NREFLOW
- added R22, R24: 140, Cannula_1_0:RESISTOR-0603
- added R23: 2K7, Cannula_1_0:RESISTOR-0603
- added U$5: CONN_RECT_2X3_VERT, Cannula_1_0:CONN_RECT_2X3_VERT
- added U$7, U$9: SHORT, Cannula_1_0:SHORT
- M1, M2, M3, M4, M5, M6: value LED_R -> LED_G
- R10, R11, R12, R13, R14, R15: value 150 -> 140
- R8, R9: value 2.7k -> 2K7
- STATUS_M1, STATUS_M2, STATUS_M3, STATUS_M4, STATUS_M5, STATUS_M6: value LED_G -> LED_B
Connections:
- net ENABLE_GLOBAL renamed GLOBAL_INHIBIT
- net N$17 renamed T_VIN
- net N$25 renamed VUSB
- removed net I2C_GP1: I2C_GPIO.GP1, TP10.TP
- new net B: Q1.G, R22.1
- new net C: INHIBIT.C, Q1.D
- new net I2C_LED: I2C_GPIO.GP1, LED_DRIVER2.I7
- new net N$16: MOT4.A12
- new net N$17: ERROR.A, R24.1
- new net N$25: ERROR.C, LED_DRIVER2.O7
- new net N$26: MOT5.A12
- new net N$27: MOT2.A12
- new net N$28: MOT3.A12
- new net N$29: MOT6.A12
- new net SDO: MOT6.A5, U$9.P$1
- new net T_A12: TEENSY3.2.A12, U$5.2
- net 3.3V: now also U$5.5
- net 5V: now also R24.2
- net BRAKE_HW: now also R22.2; no longer LED_DRIVER1.I7
- net GND: now also Q1.S, R23.2, U$5.3, Y1GND.GND; no longer R18.2
- net MISO: now also U$9.P$2; no longer MOT6.A5
- net MOSI: now also U$7.P$2
- net N$11: now also MOT1.A12; no longer ENABLE_GLOBAL.C, LED_DRIVER1.O7
- net N$5: now also INHIBIT.A; no longer ENABLE_GLOBAL.A
- net SDI01: now also U$7.P$1
- net T_A10: now also R18.2, R23.1, U$5.6
- net T_A11: now also U$5.4
- net T_A13: now also U$5.1
- net XA: now also Y1G$1.2; no longer Y1.2
- net XB: now also Y1G$1.1; no longer Y1.1
Other:
- note added: "For 24V max -> use 2K7 resistor Vin = Vout * (10K + 2K7)/2K7 + 10V = Vout * 4.704 + 10 For 36V max -> use 1K resistor Vin = Vout * 11.0 + 10"
- note added: "Input Voltage Monitor:"
- moved on the sheet: C3, C4, C5, CLOCKGEN, CY, D1, D2, D3, DCDC-5V, DOWN, E-STOP, F1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

Commit message: Finished edits
Parts:
- removed CY: 100nF, SparkFun-Capacitors:CAP0603-CAP
- removed INHIBIT: LED_R, Cannula_1_0:LED-0805
- removed TSM150P04LCS: PMOS, SparkFun-DiscreteSemi:MOSFET-PCHANNEL-SOIC8SOIC8
- added C6: 100nF, SparkFun-Capacitors:CAP0603-CAP
- added D4: DIODE-POWERDI123, Cannula_1_0:DIODE-POWERDI123
- added Q2: (no value), adafruit:MOSFET-NREFLOW
- C1, C2: value 100nF -> 10uF; device SparkFun-Capacitors:CAP0603-CAP -> SparkFun-Passives:CAP1210
- C3, C5: value 10uF -> 100nF; device SparkFun-Passives:CAP1210 -> SparkFun-Capacitors:CAP0603-CAP
- D2: value DIODE-POWERDI123 -> LED_R; device Cannula_1_0:DIODE-POWERDI123 -> Cannula_1_0:LED-0805
- ERROR: value LED_G -> LED_R
- Q1: value (none) -> PMOS; device adafruit:MOSFET-NREFLOW -> SparkFun-DiscreteSemi:MOSFET-PCHANNEL-SOIC8SOIC8
- R1: value 33 -> 10k
- R10, R6: value 140 -> 2K7
- R16, R18, R19: value 10k -> 140
- R17, R7: value 140 -> 150
- R2: value 140 -> 33
- R21: value 150 -> 140
- R23, R8: value 2K7 -> 140
- R3, R5: value 140 -> 10k
- renumbered CLOCKGEN to U1, DCDC-5V to VR2, DOWN to B2, I2C_GPIO to U2, IA0515S to VR1, LED_DRIVER1 to IC2, LED_DRIVER2 to IC1, M1 to D6, M2 to D7, M3 to D8, M4 to D9, M5 to D10, M6 to D11, MENU to B3, MODE_MANUAL to D20, MODE_ROS to D19, MODE_SWITCH to S2, MOT1 to PCIE1, MOT2 to PCIE2, MOT3 to PCIE3, MOT4 to PCIE4, MOT5 to PCIE5, MOT6 to PCIE6, PGM to S1, POWER to D5, PWN_MAIN to JP1, STATUS_M1 to D13, STATUS_M2 to D14, STATUS_M3 to D15, STATUS_M4 to D16, STATUS_M5 to D17, STATUS_M6 to D18, TEENSY3.2 to TEENSY_3.2, U$5 to J1, U$7 to JP3, U$9 to JP4, UP to B1
Connections:
- net 3.3V: now also C3.1, C5.1, R1.2, R10.2, R3.1; no longer C4.1, CY.1, R16.2, R19.1, R8.2
- net 5V: now also C4.1, C6.1, D4.A, R16.2, R18.2, R19.2, R22.2, R23.2, R8.2; no longer C1.1, C5.1, D2.A, R10.2, R2.2, R3.2, R4.2, R5.2, R6.2
- net B: now also Q2.G, R4.1; no longer Q1.G, R22.1
- net BRAKE_HW: now also R3.2, R4.2; no longer R19.2, R22.2
- net C: now also D2.C, Q2.D; no longer INHIBIT.C, Q1.D
- net GLOBAL_INHIBIT: now also R1.1; no longer R16.1
- net GND: now also C6.2, Q2.S, R6.2; no longer CY.2, Q1.S, R23.2
- net N$12: now also R24.1; no longer R20.1
- net N$17: now also R17.1; no longer R24.1
- net N$19: now also R22.1; no longer R2.1
- net N$20: now also R18.1; no longer R3.1
- net N$21: now also R19.1; no longer R4.1
- net N$22: now also R20.1; no longer R5.1
- net N$23: now also R21.1; no longer R6.1
- net N$24: now also R23.1; no longer R7.1
- net N$5: now also D2.A, R7.1; no longer INHIBIT.A, R21.1
- net N$55: now also R15.1; no longer R10.1
- net N$6: now also Q1.G, R5.1; no longer R18.1, TSM150P04LCS.G
- net N$60: now also R16.1; no longer R15.1
- net N$8: now also Q1.D@1, Q1.D@2, Q1.D@3, Q1.D@4; no longer TSM150P04LCS.D@1, TSM150P04LCS.D@2, TSM150P04LCS.D@3, TSM150P04LCS.D@4
- net N$9: now also R8.1; no longer R17.1
- net N$99: now also R2.1; no longer R1.1
- net SCL: now also R10.1; no longer R8.1
- net SCLK: now also R2.2; no longer R1.2
- net T_A10: now also R5.2, R6.1; no longer R18.2, R23.1
- net T_VIN: now also D4.C; no longer D2.C
- net VIN: now also C1.1, Q1.S@1, Q1.S@2, Q1.S@3; no longer C3.1, TSM150P04LCS.S@1, TSM150P04LCS.S@2, TSM150P04LCS.S@3
Other:
- moved on the sheet: C1, C2, C3, C4, C5, R1, R10, R15, R16, R17, R18, R19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
